File: example/schematics/LED.kicad_sch (KiCad schematic)
At the start: 3 parts

Commit message: feat: clearer example
Parts:
- renumbered Green201 to Led201
Changed lines of the file:
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@@
 		(on_board yes)
 		(dnp no)
-		(property "Reference" "Green201"
+		(property "Reference" "Led201"
 			(at 49.53 104.14 90)
 			(effects
@@
 			(project "example"
 				(path "/5351644a-feec-44d6-96c1-fe5e2f09e3b2/5481df2f-3d1c-497f-a46e-a89035ddac91"
-					(reference "Green501")
+					(reference "Led501")
 					(unit 1)
 				)
 				(path "/5351644a-feec-44d6-96c1-fe5e2f09e3b2/55f4561b-9e3d-49cb-987f-e3c418905dc4"
-					(reference "Green201")
+					(reference "Led201")
 					(unit 1)
 				)
 				(path "/5351644a-feec-44d6-96c1-fe5e2f09e3b2/92d1b184-642b-4766-91b4-271674e56d9a"
-					(reference "Green301")
+					(reference "Led301")
 					(unit 1)
 				)
 				(path "/5351644a-feec-44d6-96c1-fe5e2f09e3b2/9310c729-f6b0-410f-86e8-d02638b9425f"
-					(reference "Green601")
+					(reference "Led601")
 					(unit 1)
 				)
 				(path "/5351644a-feec-44d6-96c1-fe5e2f09e3b2/dca69bc7-b3d7-495f-af05-33d03983af18"
-					(reference "Green401")
+					(reference "Led401")
 					(unit 1)
 				)
